Commit message: kuka moved + ee

File: dynamics/kuka/kuka.urdf (robot description, URDF)
Before this commit: robot iiwa14, 11 links, 10 joints
Joints:
- joint base_joint: origin xyz=0 0 0.0 rpy=0 0 0 -> xyz=-2.66 0 0.0 rpy=0 0 0

File: dynamics/kuka/temp/kuka.urdf (robot description, URDF)
Before this commit: robot iiwa14, 11 links, 10 joints
Joints:
- joint base_joint: origin xyz=0 0 0.0 rpy=0 0 0 -> xyz=-2.66 0 0.0 rpy=0 0 0

Commit message: mini-golf kuka in progress

File: dynamics/kuka/kuka.urdf (robot description, URDF)
Before this commit: robot iiwa14, 11 links, 10 joints
Joints:
- joint base_joint: origin xyz=-2.66 0 0.0 rpy=0 0 0 -> xyz=0.0 2.5 0.0 rpy=0 0 0

File: dynamics/kuka/temp/kuka.urdf (robot description, URDF)
Before this commit: robot iiwa14, 11 links, 10 joints
Joints:
- joint base_joint: origin xyz=-2.66 0 0.0 rpy=0 0 0 -> xyz=0.0 2.5 0.0 rpy=0 0 0

Commit message: weird issues

File: dynamics/kuka/kuka.urdf (robot description, URDF)
Before this commit: robot iiwa14, 11 links, 10 joints
Joints:
- joint base_joint: origin xyz=0.0 2.5 0.0 rpy=0 0 0 -> xyz=0.0 2.67 0.0 rpy=0 0 0

File: dynamics/kuka/temp/kuka.urdf (robot description, URDF)
Before this commit: robot iiwa14, 11 links, 10 joints
Joints:
- joint base_joint: origin xyz=0.0 2.5 0.0 rpy=0 0 0 -> xyz=0.0 2.67 0.0 rpy=0 0 0

Commit message: kuka mini golf working

File: dynamics/kuka/kuka.urdf (robot description, URDF)
Before this commit: robot iiwa14, 11 links, 10 joints
Joints:
- joint base_joint: origin xyz=0.0 2.67 0.0 rpy=0 0 0 -> xyz=0.0 0.0 0.0 rpy=0 0 0

File: dynamics/kuka/temp/kuka.urdf (robot description, URDF)
Before this commit: robot iiwa14, 11 links, 10 joints
Joints:
- joint base_joint: origin xyz=0.0 2.67 0.0 rpy=0 0 0 -> xyz=0.0 0.0 0.0 rpy=0 0 0
