Commit message: implicit midpoint integration, sample objective change

File: dynamics/biped/urdf/flip_5link_fromrightfoot.urdf (robot description, URDF)
Before this commit: robot flip_5link, 6 links, 5 joints
Joints:
- joint world_joint: origin xyz=0.0 0.0 0.0 rpy=0.0 0.0 0.0 -> xyz=0.21949 -.44 0.0 rpy=0.0 0.0 0.0

Commit message: 2 step animation

File: dynamics/biped/urdf/flip_5link_fromrightfoot.urdf (robot description, URDF)
Before this commit: robot flip_5link, 6 links, 5 joints
Joints:
- joint world_joint: origin xyz=0.21949 -.44 0.0 rpy=0.0 0.0 0.0 -> xyz=0.1163 -.44 0.0 rpy=0.0 0.0 0.0
